Commit message: Add hand-camera calibration

File: frcobot_description/urdf/fr10_gazebo.urdf (robot description, URDF)
Before this commit: robot FR10-V5.0.SLDASM, 17 links, 16 joints
Links:
- added link realsense_calib_link, mass 0.001
Joints:
- added joint realsense_calib_joint: type fixed, parent wrist3_Link, child realsense_calib_link, origin xyz=-0.06 0.08 0 rpy=0 0 0

File: frcobot_description/urdf/fr10_robot.urdf (robot description, URDF)
Before this commit: robot FR10-V5.0.SLDASM, 9 links, 8 joints
Links:
- added link realsense_calib_link, mass 0.001
Joints:
- added joint realsense_calib_joint: type fixed, parent wrist3_Link, child realsense_calib_link, origin xyz=-0.06 0.08 0 rpy=0 0 0

Commit message: update with moveit_callibarion module

File: frcobot_description/urdf/fr10_gazebo.urdf (robot description, URDF)
Before this commit: robot FR10-V5.0.SLDASM, 18 links, 17 joints
Links:
- added link marker_link, mass 0.14186; collision box size=0.008 0.05 0.2; collision box size=0.008 0.05 0.2
Joints:
- added joint marker_joint: type fixed, parent wrist3_Link, child marker_link, origin xyz=0 0.08 0 rpy=-1.57 0 1.57

Commit message: fix octomap

File: frcobot_description/urdf/fr10_gazebo.urdf (robot description, URDF)
Before this commit: robot FR10-V5.0.SLDASM, 19 links, 18 joints
Links:
- removed link ground_plane_box
Joints:
- removed joint ground_plane_box

Commit message: Add interations module

File: frcobot_description/urdf/fr10_gazebo.urdf (robot description, URDF)
Before this commit: robot FR10-V5.0.SLDASM, 18 links, 17 joints
Links:
- added link ground_plane_box; collision box size=10.0 10.0 0.005; visual box size=10.0 10.0 0.005
Joints:
- added joint ground_plane_box: type fixed, parent world, child ground_plane_box, origin xyz=0 0 -0.005 rpy=0 0 0
